File: WBA/Input_Amp.kicad_sch (KiCad schematic)
At the start: 36 parts, among them J1 Signal input, J17 Amp Selector, J19 Detector Input, U12 TL072, U21 OP07BRZ, U22 OP07BRZ, U23 INA128, U24 INA128

Commit message: design submitted to jlc
Parts:
- removed TP2: TestPoint0, TestPoint:TestPoint_Loop_D2.54mm_Drill1.5mm_Beaded, symbol Connector:TestPoint
- removed TP3: TestPoint1, TestPoint:TestPoint_Loop_D2.54mm_Drill1.5mm_Beaded, symbol Connector:TestPoint
