File: WBA/WBA.kicad_sch (KiCad schematic)
At the start: 79 parts, among them J10 Conn_01x02, J11 Conn_01x02, J12 Conn_01x02, J13 Conn_01x02, J14 Conn_01x02, J15 Conn_01x02, J16 LPF_potentiometer_100k, J2 Conn_01x24, J3 Conn_01x04, J4 Conn_01x24, J6 Conn_01x04, J7 Conn_01x04, J8 Conn_01x02, J9 Conn_01x02, U1 Teensy4.1, U11 MAX7424EUA+T, U19 TLV2374IDR, U2 TLV2372, U20 TLV2374IDR, U3 MAX7424EUA+T

Commit message: more compact layout
Parts:
- C10, C13, C16, C19, C9: footprint Capacitor_SMD:C_0402_1005Metric -> Capacitor_SMD:C_0603_1608Metric; LCSC C1518204 -> C53987
- C39, C40, C41, C42, C43, C46, C47: footprint Capacitor_SMD:C_0402_1005Metric -> Capacitor_SMD:C_0603_1608Metric; LCSC C1525 -> C14663
Changed lines of the file:
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@@
 			)
 		)
-		(property "Footprint" "Capacitor_SMD:C_0402_1005Metric"
+		(property "Footprint" "Capacitor_SMD:C_0603_1608Metric"
 			(at 66.04 68.8848 0)
 			(hide yes)
@@
 			)
 		)
-		(property "LCSC" "C1518204"
+		(property "LCSC" "C53987"
 			(at 62.23 69.85 90)
 			(hide yes)
@@
 			)
 		)
-		(property "Footprint" "Capacitor_SMD:C_0402_1005Metric"
+		(property "Footprint" "Capacitor_SMD:C_0603_1608Metric"
 			(at 63.5 134.9248 0)
 			(hide yes)
@@
 			)
 		)
-		(property "LCSC" "C1518204"
+		(property "LCSC" "C53987"
 			(at 59.69 135.89 90)
 			(hide yes)
@@
 			)
 		)
-		(property "Footprint" "Capacitor_SMD:C_0402_1005Metric"
+		(property "Footprint" "Capacitor_SMD:C_0603_1608Metric"
 			(at 66.04 34.5948 0)
 			(hide yes)
@@
 			)
 		)
-		(property "LCSC" "C1518204"
+		(property "LCSC" "C53987"
 			(at 62.23 35.56 90)
 			(hide yes)
@@
 			)
 		)
-		(property "Footprint" "Capacitor_SMD:C_0402_1005Metric"
+		(property "Footprint" "Capacitor_SMD:C_0603_1608Metric"
 			(at 266.3952 78.74 0)
 			(hide yes)
@@
 			)
 		)
-		(property "LCSC" "C1525"
+		(property "LCSC" "C14663"
 			(at 265.43 74.93 0)
 			(hide yes)
@@
 			)
 		)
-		(property "Footprint" "Capacitor_SMD:C_0402_1005Metric"
+		(property "Footprint" "Capacitor_SMD:C_0603_1608Metric"
 			(at 122.2248 29.21 0)
 			(hide yes)
@@
 			)
 		)
-		(property "LCSC" "C1525"
+		(property "LCSC" "C14663"
 			(at 123.19 25.4 0)
 			(hide yes)
@@
 			)
 		)
-		(property "Footprint" "Capacitor_SMD:C_0402_1005Metric"
+		(property "Footprint" "Capacitor_SMD:C_0603_1608Metric"
 			(at 296.2148 55.88 0)
 			(hide yes)
@@
 			)
 		)
-		(property "LCSC" "C1525"
+		(property "LCSC" "C14663"
 			(at 297.18 52.07 0)
 			(hide yes)
@@
 			)
 		)
-		(property "Footprint" "Capacitor_SMD:C_0402_1005Metric"
+		(property "Footprint" "Capacitor_SMD:C_0603_1608Metric"
 			(at 266.3952 125.73 0)
 			(hide yes)
@@
 			)
 		)
-		(property "LCSC" "C1525"
+		(property "LCSC" "C14663"
 			(at 265.43 121.92 0)
 			(hide yes)
@@
 			)
 		)
-		(property "Footprint" "Capacitor_SMD:C_0402_1005Metric"
+		(property "Footprint" "Capacitor_SMD:C_0603_1608Metric"
 			(at 155.2448 29.21 0)
 			(hide yes)
@@
 			)
 		)
-		(property "LCSC" "C1525"
+		(property "LCSC" "C14663"
 			(at 156.21 25.4 0)
 			(hide yes)
@@
 			)
 		)
-		(property "Footprint" "Capacitor_SMD:C_0402_1005Metric"
+		(property "Footprint" "Capacitor_SMD:C_0603_1608Metric"
 			(at 296.2148 104.14 0)
 			(hide yes)
@@
 			)
 		)
-		(property "LCSC" "C1525"
+		(property "LCSC" "C14663"
 			(at 297.18 100.33 0)
 			(hide yes)
@@
 			)
 		)
-		(property "Footprint" "Capacitor_SMD:C_0402_1005Metric"
+		(property "Footprint" "Capacitor_SMD:C_0603_1608Metric"
 			(at 63.5 162.8648 0)
 			(hide yes)
@@
 			)
 		)
-		(property "LCSC" "C1518204"
+		(property "LCSC" "C53987"
 			(at 59.69 163.83 90)
 			(hide yes)
@@
 			)
 		)
-		(property "Footprint" "Capacitor_SMD:C_0402_1005Metric"
+		(property "Footprint" "Capacitor_SMD:C_0603_1608Metric"
 			(at 55.88 103.1748 0)
 			(hide yes)
@@
 			)
 		)
-		(property "LCSC" "C1518204"
+		(property "LCSC" "C53987"
 			(at 59.69 104.14 90)
 			(hide yes)
@@
 			)
 		)
-		(property "Footprint" "Capacitor_SMD:C_0402_1005Metric"
+		(property "Footprint" "Capacitor_SMD:C_0603_1608Metric"
 			(at 336.2452 26.67 0)
 			(hide yes)
@@
 			)
 		)
-		(property "LCSC" "C1525"
+		(property "LCSC" "C14663"
 			(at 335.28 22.86 0)
 			(hide yes)

Commit message: design submitted to jlc
Parts:
- removed U11, U3: MAX7424EUA+T, Package_SO:MSOP-8_3x3mm_P0.65mm, symbol Filter:MAX7424xUA
- added U3, U4: MAX7414xUA, Package_SO:MSOP-8_3x3mm_P0.65mm, symbol Filter:MAX7414xUA
Connections:
- net +3.3V: now also U3.4 (V_{DD}), U3.7 (~{SHDN}), U4.4 (V_{DD}), U4.7 (~{SHDN})
- net GND: now also U3.3 (GND), U4.3 (GND)
- net at C3.1, R6.1: now also U3.2 (IN)
- net at C41.1: now also U4.1 (COM), U4.6 (OS)
- net at C42.1: now also U3.1 (COM), U3.6 (OS)
- net at R35.2: now also U3.5 (OUT)
- net at J4.21 (Pin_21): now also U3.8 (CLK), U4.8 (CLK)
- net at C1.1, R3.1: now also U4.2 (IN)
- net at R34.2: now also U4.5 (OUT)
