File: WBA/power.kicad_sch (KiCad schematic)
At the start: 28 parts, among them J5 Input Power, Q1 A03400A, Q2 A03401A, U14 L7805, U15 L7905, U16 TPS5430DDA, U8 L7805

Commit message: more compact layout
Parts:
- removed D3, D7: 1N4148, Diode_THT:D_DO-35_SOD27_P7.62mm_Horizontal, symbol Diode:1N4148
- added D1, D2: 1N4148W, Diode_SMD:D_SOD-123, symbol Diode:1N4148W
- C29, C81: footprint Capacitor_SMD:C_0402_1005Metric -> Capacitor_SMD:C_0603_1608Metric; LCSC C1525 -> C14663
- C30: footprint Capacitor_SMD:C_0402_1005Metric -> Capacitor_SMD:C_0603_1608Metric; LCSC C15195 -> C57112
Connections:
- net at Q2.1 (G), R36.1: now also D1.2 (A)
- net at C28.1, C54.1, C83.1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: now also D1.1 (K)
- net at Q1.1 (G), R38.1: now also D2.1 (K)
- net at C73.2, Q1.2 (S), R40.1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: now also D2.2 (A)

Commit message: design submitted to jlc
Parts:
- C30: value 0.01uF -> 10nF
- C31: LCSC C72494 -> C2833309
- D1, D2: LCSC (none) -> C81598
- U16: LCSC C2886400 -> C9864
Changed lines of the file:
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@@
 			)
 		)
+		(property "LCSC" "C81598"
+			(at 88.9 170.18 0)
+			(hide yes)
+			(show_name no)
+			(do_not_autoplace no)
+			(effects
+				(font
+					(size 1.27 1.27)
+				)
+			)
+		)
 		(pin "2"
 		)
@@
 			)
 		)
-		(property "Value" "0.01uF"
+		(property "Value" "10nF"
 			(at 190.5 52.07 90)
 			(show_name no)
@@
 			)
 		)
-		(property "LCSC" "C2886400"
+		(property "LCSC" "C9864"
 			(at 171.45 62.23 0)
 			(hide yes)
@@
 			)
 		)
+		(property "LCSC" "C81598"
+			(at 88.9 90.17 0)
+			(hide yes)
+			(show_name no)
+			(do_not_autoplace no)
+			(effects
+				(font
+					(size 1.27 1.27)
+				)
+			)
+		)
 		(pin "2"
 		)
@@
 			)
 		)
-		(property "LCSC" "C72494"
+		(property "LCSC" "C2833309"
 			(at 209.55 60.96 0)
 			(hide yes)
